File: TapecartFlasher.sch (KiCad schematic (older format))
At the start: 18 parts, among them J1 C64-CassettePort, P1 Digital, P2 Analog, P3 CONN_01X01, P4 CONN_01X01, P5 CONN_01X01, P6 CONN_01X01, Q1 BC547, Q2 BC557

Commit message: Added SD module connector and motor voltage jumper.
Parts:
- added J2: SD Module, Socket_Strips:Socket_Strip_Angled_1x06_Pitch2.54mm, symbol Connector:Conn_01x06_Female
- added JP1: Vmotor, Pin_Headers:Pin_Header_Straight_1x03_Pitch2.54mm, symbol w_conn:GS3
Connections:
- net labels added: SD_MISO, SD_MOSI, SD_SCK, SD_SEL
- wire segments 88 -> 92
Changed lines of the file:
@@
 encoding utf-8
 Sheet 1 1
-Title ""
-Date "jeu. 02 avril 2015"
-Rev ""
-Comp ""
+Title "TapecartFlasher"
+Date "2018-08-26"
+Rev "Rev.1"
+Comp "hackup.net"
 Comment1 ""
 Comment2 ""
@@
 Text Label 8700 2500 0    60   ~ 0
 12(MISO)
-Text Label 10550 2500 0    60   ~ 0
+Text Label 10150 2500 0    60   ~ 0
 13(SCK)
 Text Label 10550 2200 0    60   ~ 0
@@
 	2500 2200 2500 1650
 Connection ~ 2500 1650
-Wire Wire Line
-	2500 1650 2800 1650
 Text GLabel 8700 1500 0    50   Input ~ 0
 Motor5
@@
 Text GLabel 8700 1800 0    50   Input ~ 0
 Sense
-Text GLabel 2800 1650 2    50   Input ~ 0
+Text GLabel 3350 1550 2    50   Input ~ 0
 Motor7
 Text GLabel 2800 1750 2    50   Input ~ 0
@@
 Wire Wire Line
 	5650 2550 6000 2550
+$Comp
+L Connector:Conn_01x06_Female J2
+U 1 1 5B831172
+P 8600 4000
+F 0 "J2" H 8627 3976 50  0000 L CNN
+F 1 "SD Module" H 8627 3885 50  0000 L CNN
+F 2 "Socket_Strips:Socket_Strip_Angled_1x06_Pitch2.54mm" H 8600 4000 50  0001 C CNN
+F 3 "~" H 8600 4000 50  0001 C CNN
+	1    8600 4000
+	1    0    0    -1
+$EndComp
+Text GLabel 8400 4000 0    50   Input ~ 0
+SD_MISO
+Text GLabel 8400 4100 0    50   Input ~ 0
+SD_MOSI
+Text GLabel 8400 4200 0    50   Input ~ 0
+SD_SCK
+Text GLabel 8400 4300 0    50   Input ~ 0
+SD_SEL
+$Comp
+L power:GND #PWR0108
+U 1 1 5B8315FA
+P 7900 4450
+F 0 "#PWR0108" H 7900 4200 50  0001 C CNN
+F 1 "GND" H 7900 4300 50  0000 C CNN
+F 2 "" H 7900 4450 50  0000 C CNN
+F 3 "" H 7900 4450 50  0000 C CNN
+	1    7900 4450
+	1    0    0    -1
+$EndComp
+Wire Wire Line
+	8400 3800 7900 3800
+Wire Wire Line
+	7900 3800 7900 4450
+$Comp
+L power:+5V #PWR0109
+U 1 1 5B8343B1
+P 8000 3700
+F 0 "#PWR0109" H 8000 3550 50  0001 C CNN
+F 1 "+5V" H 8000 3840 28  0000 C CNN
+F 2 "" H 8000 3700 50  0000 C CNN
+F 3 "" H 8000 3700 50  0000 C CNN
+	1    8000 3700
+	1    0    0    -1
+$EndComp
+Wire Wire Line
+	8400 3900 8000 3900
+Wire Wire Line
+	8000 3900 8000 3700
+Text GLabel 8700 2300 0    50   Input ~ 0
+SD_SEL
+Text GLabel 8700 2400 0    50   Input ~ 0
+SD_MOSI
+Text GLabel 8700 2500 0    50   Input ~ 0
+SD_MISO
+Text GLabel 10550 2500 2    50   Input ~ 0
+SD_SCK
+$Comp
+L w_conn:GS3 JP1
+U 1 1 5B8479B7
+P 3200 1650
+F 0 "JP1" H 3200 1361 50  0000 C CNN
+F 1 "Vmotor" H 3200 1445 40  0000 C CNN
+F 2 "Pin_Headers:Pin_Header_Straight_1x03_Pitch2.54mm" H 3200 1650 50  0001 C CNN
+F 3 "" H 3200 1650 50  0001 C CNN
+	1    3200 1650
+	-1   0    0    1
+$EndComp
+Text GLabel 3350 1750 2    50   Input ~ 0
+Motor5
+Wire Wire Line
+	2500 1650 3050 1650
 $EndSCHEMATC

Commit message: Preparing for Gerber export.
Parts:
- removed P3, P4, P5, P6: CONN_01X01, Socket_Arduino_Nano:1pin_Nano, symbol TapecartFlasher-rescue:CONN_01X01
- JP1: symbol w_conn:GS3 -> conn:GS3
Connections:
- no-connect marks 4 -> 0
Other:
- note removed: "Holes"
Changed lines of the file:
@@
 Text Label 10550 1300 0    60   ~ 0
 RST
-Text Notes 10800 1000 0    60   ~ 0
-Holes
 Text Notes 8350 575  0    60   ~ 0
 Shield for Arduino Nano
@@
 Wire Notes Line
 	9525 650  9525 475
-$Comp
-L TapecartFlasher-rescue:CONN_01X01 P3
-U 1 1 56D73ADD
-P 10800 650
-F 0 "P3" V 10900 650 50  0000 C CNN
-F 1 "CONN_01X01" V 10900 650 50  0001 C CNN
-F 2 "Socket_Arduino_Nano:1pin_Nano" H 10800 650 50  0001 C CNN
-F 3 "" H 10800 650 50  0000 C CNN
-	1    10800 650
-	0    -1   -1   0
-$EndComp
-NoConn ~ 10800 850
-$Comp
-L TapecartFlasher-rescue:CONN_01X01 P4
-U 1 1 56D73D86
-P 10900 650
-F 0 "P4" V 11000 650 50  0000 C CNN
-F 1 "CONN_01X01" V 11000 650 50  0001 C CNN
-F 2 "Socket_Arduino_Nano:1pin_Nano" H 10900 650 50  0001 C CNN
-F 3 "" H 10900 650 50  0000 C CNN
-	1    10900 650
-	0    -1   -1   0
-$EndComp
-$Comp
-L TapecartFlasher-rescue:CONN_01X01 P5
-U 1 1 56D73DAE
-P 11000 650
-F 0 "P5" V 11100 650 50  0000 C CNN
-F 1 "CONN_01X01" V 11100 650 50  0001 C CNN
-F 2 "Socket_Arduino_Nano:1pin_Nano" H 11000 650 50  0001 C CNN
-F 3 "" H 11000 650 50  0000 C CNN
-	1    11000 650
-	0    -1   -1   0
-$EndComp
-$Comp
-L TapecartFlasher-rescue:CONN_01X01 P6
-U 1 1 56D73DD9
-P 11100 650
-F 0 "P6" V 11200 650 50  0000 C CNN
-F 1 "CONN_01X01" V 11200 650 50  0001 C CNN
-F 2 "Socket_Arduino_Nano:1pin_Nano" H 11100 650 50  0001 C CNN
-F 3 "" H 11100 650 50  0000 C CNN
-	1    11100 650
-	0    -1   -1   0
-$EndComp
-NoConn ~ 10900 850
-NoConn ~ 11000 850
-NoConn ~ 11100 850
 $Comp
 L TapecartFlasher-rescue:CONN_01X15 P1
@@
 Wire Wire Line
 	10150 2500 10550 2500
-Wire Notes Line
-	11200 1050 10650 1050
-Wire Notes Line
-	10650 1050 10650 500
 Wire Notes Line
 	11150 2850 8400 2850
@@
 SD_SCK
 $Comp
-L w_conn:GS3 JP1
+L conn:GS3 JP1
 U 1 1 5B8479B7
 P 3200 1650

Commit message: Annotated schematics.
Other:
- note added: "Cassete Port Connector"
- note added: "Charge Pump and Motor Signal"
- note added: "SD Module Connector"
Changed lines of the file:
@@
 Wire Wire Line
 	10150 2500 10550 2500
-Wire Notes Line
-	11150 2850 8400 2850
-Wire Notes Line
-	8300 2850 8300 500
 Text Notes 9650 1100 0    60   ~ 0
 1
@@
 Wire Wire Line
 	2500 1650 3050 1650
+Wire Notes Line
+	900  700  900  3700
+Wire Notes Line
+	900  3700 3800 3700
+Wire Notes Line
+	3800 3700 3800 700
+Wire Notes Line
+	900  700  3800 700
+Wire Notes Line
+	3950 700  3950 3700
+Wire Notes Line
+	3950 3700 7150 3700
+Wire Notes Line
+	7150 3700 7150 700
+Wire Notes Line
+	7150 700  3950 700
+Wire Notes Line
+	7600 3350 7600 4900
+Wire Notes Line
+	7600 4900 9550 4900
+Wire Notes Line
+	9550 4900 9550 3350
+Wire Notes Line
+	9550 3350 7600 3350
+Wire Notes Line
+	8300 500  8300 2850
+Wire Notes Line
+	8300 2850 11200 2850
+Text Notes 8500 4850 0    60   ~ 0
+SD Module Connector
+Text Notes 5650 3650 0    60   ~ 0
+Charge Pump and Motor Signal
+Text Notes 2650 3650 0    60   ~ 0
+Cassete Port Connector
 $EndSCHEMATC

Commit message: Changed resistor footprints.
Parts:
- D3: value 7.5 -> 6.8
- JP1: symbol conn:GS3 -> w_conn:GS3
- Q1, Q2: footprint TO_SOT_Packages_THT:TO-92_Inline_Narrow_Oval -> TO_SOT_Packages_THT:TO-92_Molded_Narrow
Changed lines of the file:
@@
 P 6250 1850
 F 0 "D3" V 6204 1929 50  0000 L CNN
-F 1 "7.5" V 6295 1929 50  0000 L CNN
+F 1 "6.8" V 6295 1929 50  0000 L CNN
 F 2 "Diodes_THT:D_T-1_P5.08mm_Horizontal" H 6250 1850 50  0001 C CNN
 F 3 "https://en.wikipedia.org/wiki/Zener_diode" H 6250 1850 50  0001 C CNN
@@
 F 0 "Q2" H 6091 2854 50  0000 L CNN
 F 1 "BC557" H 6091 2945 50  0000 L CNN
-F 2 "TO_SOT_Packages_THT:TO-92_Inline_Narrow_Oval" H 6100 2825 50  0001 L CIN
+F 2 "TO_SOT_Packages_THT:TO-92_Molded_Narrow" H 6100 2825 50  0001 L CIN
 F 3 "http://www.fairchildsemi.com/ds/BC/BC557.pdf" H 5900 2900 50  0001 L CNN
 	1    5900 2900
@@
 F 0 "Q1" H 5341 3196 50  0000 L CNN
 F 1 "BC547" H 5341 3105 50  0000 L CNN
-F 2 "TO_SOT_Packages_THT:TO-92_Inline_Narrow_Oval" H 5350 3075 50  0001 L CIN
+F 2 "TO_SOT_Packages_THT:TO-92_Molded_Narrow" H 5350 3075 50  0001 L CIN
 F 3 "http://www.fairchildsemi.com/ds/BC/BC547.pdf" H 5150 3150 50  0001 L CNN
 	1    5150 3150
@@
 SD_SCK
 $Comp
-L conn:GS3 JP1
+L w_conn:GS3 JP1
 U 1 1 5B8479B7
 P 3200 1650

Commit message: Modified/corrected zender diode circuit.
Parts:
- JP1: symbol w_conn:GS3 -> conn:GS3
Connections:
- wire segments 92 -> 95
Changed lines of the file:
@@
 Sheet 1 1
 Title "TapecartFlasher Nano"
-Date "2018-08-26"
-Rev "Rev.1"
+Date "2018-09-06"
+Rev "Rev.2"
 Comp "hackup.net"
 Comment1 ""
@@
 L device:R R1
 U 1 1 5B665553
-P 6250 1550
-F 0 "R1" V 6043 1550 50  0000 C CNN
-F 1 "10" V 6134 1550 50  0000 C CNN
-F 2 "Resistors_THT:R_Axial_DIN0207_L6.3mm_D2.5mm_P7.62mm_Horizontal" V 6180 1550 50  0001 C CNN
-F 3 "" H 6250 1550 50  0001 C CNN
-	1    6250 1550
-	-1   0    0    1
+P 5950 1400
+F 0 "R1" V 5743 1400 50  0000 C CNN
+F 1 "10" V 5834 1400 50  0000 C CNN
+F 2 "Resistors_THT:R_Axial_DIN0207_L6.3mm_D2.5mm_P7.62mm_Horizontal" V 5880 1400 50  0001 C CNN
+F 3 "" H 5950 1400 50  0001 C CNN
+	1    5950 1400
+	0    -1   -1   0
 $EndComp
 $Comp
 L device:D_Zener D3
 U 1 1 5B6656B6
-P 6250 1850
-F 0 "D3" V 6204 1929 50  0000 L CNN
-F 1 "6.8" V 6295 1929 50  0000 L CNN
-F 2 "Diodes_THT:D_T-1_P5.08mm_Horizontal" H 6250 1850 50  0001 C CNN
-F 3 "https://en.wikipedia.org/wiki/Zener_diode" H 6250 1850 50  0001 C CNN
-	1    6250 1850
+P 6300 1650
+F 0 "D3" V 6254 1729 50  0000 L CNN
+F 1 "6.8" V 6345 1729 50  0000 L CNN
+F 2 "Diodes_THT:D_T-1_P5.08mm_Horizontal" H 6300 1650 50  0001 C CNN
+F 3 "https://en.wikipedia.org/wiki/Zener_diode" H 6300 1650 50  0001 C CNN
+	1    6300 1650
 	0    1    1    0
 $EndComp
@@
 Wire Wire Line
 	5550 1500 5550 1400
-Connection ~ 5550 1400
 $Comp
 L power:GND #PWR0103
@@
 $EndComp
 Wire Wire Line
-	5550 1400 6250 1400
-Wire Wire Line
 	5550 1800 5550 2000
 Connection ~ 5550 2000
-Connection ~ 6250 1400
-Wire Wire Line
-	5550 2000 6250 2000
-Wire Wire Line
-	6250 1400 6750 1400
 $Comp
 L Transistor:BC557 Q2
@@
 SD_SCK
 $Comp
-L w_conn:GS3 JP1
+L conn:GS3 JP1
 U 1 1 5B8479B7
 P 3200 1650
@@
 Text Notes 2650 3650 0    60   ~ 0
 Cassete Port Connector
+Wire Wire Line
+	5550 1400 5800 1400
+Connection ~ 5550 1400
+Wire Wire Line
+	6100 1400 6300 1400
+Wire Wire Line
+	6300 1500 6300 1400
+Connection ~ 6300 1400
+Wire Wire Line
+	6300 1400 6750 1400
+Wire Wire Line
+	6300 2000 6300 1800
+Wire Wire Line
+	5550 2000 6300 2000
 $EndSCHEMATC

Commit message: Added decoupling capacitor to prevent Arduino from rebooting.
Parts:
- added C3: 220µ, Capacitors_THT:CP_Radial_D6.3mm_P2.50mm, symbol device:CP
- JP1: symbol conn:GS3 -> w_conn:GS3
Connections:
- net labels removed: +3.3V
- wire segments 95 -> 94
- no-connect marks 0 -> 18
Changed lines of the file:
@@
 Wire Wire Line
 	8700 2500 9350 2500
-$Comp
-L power:GND #PWR02
-U 1 1 56D746ED
-P 10250 2600
-F 0 "#PWR02" H 10250 2350 50  0001 C CNN
-F 1 "GND" H 10250 2450 50  0000 C CNN
-F 2 "" H 10250 2600 50  0000 C CNN
-F 3 "" H 10250 2600 50  0000 C CNN
-	1    10250 2600
-	1    0    0    -1
-$EndComp
 Wire Wire Line
 	10250 2600 10250 1200
@@
 P 10350 950
 F 0 "#PWR03" H 10350 800 50  0001 C CNN
-F 1 "+5V" H 10350 1090 28  0000 C CNN
-F 2 "" H 10350 950 50  0000 C CNN
-F 3 "" H 10350 950 50  0000 C CNN
+F 1 "+5V" H 10350 1090 50  0000 C CNN
+F 2 "" H 10350 950 50  0001 C CNN
+F 3 "" H 10350 950 50  0001 C CNN
 	1    10350 950
 	1    0    0    -1
@@
 Wire Wire Line
 	10350 1400 10150 1400
-$Comp
-L power:+3.3V #PWR04
-U 1 1 56D74854
-P 10450 950
-F 0 "#PWR04" H 10450 800 50  0001 C CNN
-F 1 "+3.3V" H 10450 1090 28  0000 C CNN
-F 2 "" H 10450 950 50  0000 C CNN
-F 3 "" H 10450 950 50  0000 C CNN
-	1    10450 950
-	1    0    0    -1
-$EndComp
-Wire Wire Line
-	10450 950  10450 2400
-Wire Wire Line
-	10450 2400 10150 2400
 Wire Wire Line
 	10550 1300 10150 1300
@@
 SD_SCK
 $Comp
-L conn:GS3 JP1
+L w_conn:GS3 JP1
 U 1 1 5B8479B7
 P 3200 1650
@@
 Wire Wire Line
 	5550 2000 6300 2000
+$Comp
+L device:CP C3
+U 1 1 5BCF0BEB
+P 1300 2650
+F 0 "C3" H 1418 2696 50  0000 L CNN
+F 1 "220µ" H 1418 2605 50  0000 L CNN
+F 2 "Capacitors_THT:CP_Radial_D6.3mm_P2.50mm" H 1338 2500 50  0001 C CNN
+F 3 "" H 1300 2650 50  0001 C CNN
+	1    1300 2650
+	1    0    0    -1
+$EndComp
+$Comp
+L power:+5V #PWR0110
+U 1 1 5BCF0CE5
+P 1300 2500
+F 0 "#PWR0110" H 1300 2350 50  0001 C CNN
+F 1 "+5V" H 1300 2640 28  0000 C CNN
+F 2 "" H 1300 2500 50  0000 C CNN
+F 3 "" H 1300 2500 50  0000 C CNN
+	1    1300 2500
+	1    0    0    -1
+$EndComp
+$Comp
+L power:GND #PWR0111
+U 1 1 5BCF0D12
+P 1300 2800
+F 0 "#PWR0111" H 1300 2550 50  0001 C CNN
+F 1 "GND" H 1300 2650 50  0000 C CNN
+F 2 "" H 1300 2800 50  0000 C CNN
+F 3 "" H 1300 2800 50  0000 C CNN
+	1    1300 2800
+	1    0    0    -1
+$EndComp
+NoConn ~ 8700 1100
+NoConn ~ 8700 1200
+NoConn ~ 8700 1300
+NoConn ~ 8700 1900
+NoConn ~ 8700 2000
+NoConn ~ 8700 2100
+NoConn ~ 10250 950
+NoConn ~ 10550 2300
+NoConn ~ 10550 2200
+NoConn ~ 10550 2100
+NoConn ~ 10550 2000
+NoConn ~ 10550 1900
+NoConn ~ 10550 1800
+NoConn ~ 10550 1700
+NoConn ~ 10550 1600
+NoConn ~ 10550 1500
+NoConn ~ 10550 1300
+Wire Wire Line
+	9250 2600 10250 2600
+Connection ~ 9250 2600
+$Comp
+L power:PWR_FLAG #FLG0101
+U 1 1 5BD31CB6
+P 11000 850
+F 0 "#FLG0101" H 11000 925 50  0001 C CNN
+F 1 "PWR_FLAG" H 11000 1024 50  0000 C CNN
+F 2 "" H 11000 850 50  0001 C CNN
+F 3 "~" H 11000 850 50  0001 C CNN
+	1    11000 850
+	1    0    0    -1
+$EndComp
+$Comp
+L power:GND #PWR0112
+U 1 1 5BD31D0C
+P 11000 850
+F 0 "#PWR0112" H 11000 600 50  0001 C CNN
+F 1 "GND" H 11000 700 50  0000 C CNN
+F 2 "" H 11000 850 50  0000 C CNN
+F 3 "" H 11000 850 50  0000 C CNN
+	1    11000 850
+	1    0    0    -1
+$EndComp
+$Comp
+L power:+5V #PWR0113
+U 1 1 5BD31D39
+P 10700 850
+F 0 "#PWR0113" H 10700 700 50  0001 C CNN
+F 1 "+5V" H 10700 990 28  0000 C CNN
+F 2 "" H 10700 850 50  0000 C CNN
+F 3 "" H 10700 850 50  0000 C CNN
+	1    10700 850
+	1    0    0    -1
+$EndComp
+$Comp
+L power:PWR_FLAG #FLG0102
+U 1 1 5BD31D66
+P 10700 850
+F 0 "#FLG0102" H 10700 925 50  0001 C CNN
+F 1 "PWR_FLAG" H 10700 1023 50  0000 C CNN
+F 2 "" H 10700 850 50  0001 C CNN
+F 3 "~" H 10700 850 50  0001 C CNN
+	1    10700 850
+	-1   0    0    1
+$EndComp
+$Comp
+L power:PWR_FLAG #FLG0103
+U 1 1 5BD38263
+P 6900 900
+F 0 "#FLG0103" H 6900 975 50  0001 C CNN
+F 1 "PWR_FLAG" H 6900 1073 50  0000 C CNN
+F 2 "" H 6900 900 50  0001 C CNN
+F 3 "~" H 6900 900 50  0001 C CNN
+	1    6900 900
+	-1   0    0    1
+$EndComp
+$Comp
+L power:VPP #PWR0114
+U 1 1 5BD38318
+P 6900 900
+F 0 "#PWR0114" H 6900 750 50  0001 C CNN
+F 1 "VPP" H 6900 1040 28  0000 C CNN
+F 2 "" H 6900 900 50  0000 C CNN
+F 3 "" H 6900 900 50  0000 C CNN
+	1    6900 900
+	1    0    0    -1
+$EndComp
+NoConn ~ 10150 2400
 $EndSCHEMATC
